File: kb.kicad_sch (KiCad schematic)
At the start: 35 parts

Commit message: Add switches and more electronics
Parts:
- added H? (x4): MountingHole_Pad, MountingHole:MountingHole_4.3mm_M4_DIN965_Pad, symbol Mechanical:MountingHole_Pad
- C? (x2): Basic Part (none) -> Yes; LCSC part number (none) -> C7171
- J?: footprint (none) -> Connector_USB:USB_C_Receptacle_HRO_TYPE-C-31-M-12; Basic Part (none) -> No; LCSC part number (none) -> C165948
- R? (x2): Basic Part (none) -> Yes; LCSC part number (none) -> C25905
- U?: footprint RP2040_minimal:RP2040-QFN-56 -> Package_DFN_QFN:QFN-56-1EP_8x8mm_P0.5mm_EP4.3x4.3mm; Basic Part (none) -> No; LCSC part number (none) -> C2040
- U?: Basic Part (none) -> Yes; LCSC part number (none) -> C6186
- U?: Basic Part (none) -> No; LCSC part number (none) -> C2687116
Connections:
- net GND: now also H?.1, H?.1, H?.1, H?.1
- net Y3: now reaches U?.11 (GPIO8)
- net Y4: now reaches U?.12 (GPIO9)
- net Y5: now reaches U?.13 (GPIO10)
- net Y6: now reaches U?.14 (GPIO11)
- net Y7: now reaches U?.15 (GPIO12)
- net Y8: now reaches U?.16 (GPIO13)
- net Y9: now reaches U?.17 (GPIO14)
- net Y10: now reaches U?.18 (GPIO15)
- net X0: now reaches U?.2 (GPIO0)
- net Y11: now reaches U?.27 (GPIO16)
- net Y12: now reaches U?.28 (GPIO17)
- net Y13: now reaches U?.29 (GPIO18)
- net X1: now reaches U?.3 (GPIO1)
- net Y14: now reaches U?.30 (GPIO19)
- net X2: now reaches U?.4 (GPIO2)
- net X3: now reaches U?.5 (GPIO3)
- net X4: now reaches U?.6 (GPIO4)
- net Y0: now reaches U?.7 (GPIO5)
- net Y1: now reaches U?.8 (GPIO6)
- net Y2: now reaches U?.9 (GPIO7)
Other:
- note added: "+3.3V regulator"
