File: switches.kicad_sch (KiCad schematic)
At the start: 0 parts

Commit message: Add switches and more electronics
Parts:
- added C? (x2): 10nF, Capacitor_SMD:C_0402_1005Metric, symbol Device:C_Small
- added D? (x61): LL4148, Diode_SMD:D_MiniMELF, symbol Device:D_Small
- added R? (x4): 10K, Resistor_SMD:R_0402_1005Metric, symbol Device:R_Small
- added SW?: I, Button_Switch_Keyboard:SW_Cherry_MX_1.00u_PCB, symbol Switch:SW_Push
- added SW?: O, Button_Switch_Keyboard:SW_Cherry_MX_1.00u_PCB, symbol Switch:SW_Push
- added SW?: S, Button_Switch_Keyboard:SW_Cherry_MX_1.00u_PCB, symbol Switch:SW_Push
- added SW?: Backspace, Button_Switch_Keyboard:SW_Cherry_MX_1.00u_PCB, symbol Switch:SW_Push
- added SW?: ], Button_Switch_Keyboard:SW_Cherry_MX_1.00u_PCB, symbol Switch:SW_Push
- added SW?: /, Button_Switch_Keyboard:SW_Cherry_MX_1.00u_PCB, symbol Switch:SW_Push
- added SW?: 1, Button_Switch_Keyboard:SW_Cherry_MX_1.00u_PCB, symbol Switch:SW_Push
- added SW?: \, Button_Switch_Keyboard:SW_Cherry_MX_1.00u_PCB, symbol Switch:SW_Push
- added SW?: P, Button_Switch_Keyboard:SW_Cherry_MX_1.00u_PCB, symbol Switch:SW_Push
- added SW?: 5, Button_Switch_Keyboard:SW_Cherry_MX_1.00u_PCB, symbol Switch:SW_Push
- added SW?: ,, Button_Switch_Keyboard:SW_Cherry_MX_1.00u_PCB, symbol Switch:SW_Push
- added SW?: ⌄, Button_Switch_Keyboard:SW_Cherry_MX_1.00u_PCB, symbol Switch:SW_Push
- added SW?: Win, Button_Switch_Keyboard:SW_Cherry_MX_1.00u_PCB, symbol Switch:SW_Push
- added SW?: ^, Button_Switch_Keyboard:SW_Cherry_MX_1.00u_PCB, symbol Switch:SW_Push
- added SW?: Caps, Button_Switch_Keyboard:SW_Cherry_MX_1.00u_PCB, symbol Switch:SW_Push
- added SW?: [, Button_Switch_Keyboard:SW_Cherry_MX_1.00u_PCB, symbol Switch:SW_Push
- added SW?: Tab, Button_Switch_Keyboard:SW_Cherry_MX_1.00u_PCB, symbol Switch:SW_Push
- added SW?: >, Button_Switch_Keyboard:SW_Cherry_MX_1.00u_PCB, symbol Switch:SW_Push
- added SW?: -, Button_Switch_Keyboard:SW_Cherry_MX_1.00u_PCB, symbol Switch:SW_Push
- added SW?: T, Button_Switch_Keyboard:SW_Cherry_MX_1.00u_PCB, symbol Switch:SW_Push
- added SW?: `, Button_Switch_Keyboard:SW_Cherry_MX_1.00u_PCB, symbol Switch:SW_Push
- added SW? (x2): Shift, Button_Switch_Keyboard:SW_Cherry_MX_1.00u_PCB, symbol Switch:SW_Push
- added SW?: U, Button_Switch_Keyboard:SW_Cherry_MX_1.00u_PCB, symbol Switch:SW_Push
- added SW?: 8, Button_Switch_Keyboard:SW_Cherry_MX_1.00u_PCB, symbol Switch:SW_Push
- added SW?: J, Button_Switch_Keyboard:SW_Cherry_MX_1.00u_PCB, symbol Switch:SW_Push
- added SW?: F, Button_Switch_Keyboard:SW_Cherry_MX_1.00u_PCB, symbol Switch:SW_Push
- added SW?: Alt, Button_Switch_Keyboard:SW_Cherry_MX_1.00u_PCB, symbol Switch:SW_Push
- added SW?: ;, Button_Switch_Keyboard:SW_Cherry_MX_1.00u_PCB, symbol Switch:SW_Push
- added SW?: 4, Button_Switch_Keyboard:SW_Cherry_MX_1.00u_PCB, symbol Switch:SW_Push
- added SW?: R, Button_Switch_Keyboard:SW_Cherry_MX_1.00u_PCB, symbol Switch:SW_Push
- added SW?: H, Button_Switch_Keyboard:SW_Cherry_MX_1.00u_PCB, symbol Switch:SW_Push
- added SW?: 9, Button_Switch_Keyboard:SW_Cherry_MX_1.00u_PCB, symbol Switch:SW_Push
- added SW?: 7, Button_Switch_Keyboard:SW_Cherry_MX_1.00u_PCB, symbol Switch:SW_Push
- added SW?: E, Button_Switch_Keyboard:SW_Cherry_MX_1.00u_PCB, symbol Switch:SW_Push
- added SW?: M, Button_Switch_Keyboard:SW_Cherry_MX_1.00u_PCB, symbol Switch:SW_Push
- added SW?: D, Button_Switch_Keyboard:SW_Cherry_MX_1.00u_PCB, symbol Switch:SW_Push
- added SW?: G, Button_Switch_Keyboard:SW_Cherry_MX_1.00u_PCB, symbol Switch:SW_Push
- added SW?: +, Button_Switch_Keyboard:SW_Cherry_MX_1.00u_PCB, symbol Switch:SW_Push
- added SW?: Ctrl, Button_Switch_Keyboard:SW_Cherry_MX_1.00u_PCB, symbol Switch:SW_Push
- added SW?: Space, Button_Switch_Keyboard:SW_Cherry_MX_1.00u_PCB, symbol Switch:SW_Push
- added SW?: K, Button_Switch_Keyboard:SW_Cherry_MX_1.00u_PCB, symbol Switch:SW_Push
- added SW?: V, Button_Switch_Keyboard:SW_Cherry_MX_1.00u_PCB, symbol Switch:SW_Push
- added SW?: 3, Button_Switch_Keyboard:SW_Cherry_MX_1.00u_PCB, symbol Switch:SW_Push
- added SW?: Enter, Button_Switch_Keyboard:SW_Cherry_MX_1.00u_PCB, symbol Switch:SW_Push
- added SW?: X, Button_Switch_Keyboard:SW_Cherry_MX_1.00u_PCB, symbol Switch:SW_Push
- added SW?: 2, Button_Switch_Keyboard:SW_Cherry_MX_1.00u_PCB, symbol Switch:SW_Push
- added SW?: <, Button_Switch_Keyboard:SW_Cherry_MX_1.00u_PCB, symbol Switch:SW_Push
- added SW?: Z, Button_Switch_Keyboard:SW_Cherry_MX_1.00u_PCB, symbol Switch:SW_Push
- added SW?: W, Button_Switch_Keyboard:SW_Cherry_MX_1.00u_PCB, symbol Switch:SW_Push
- added SW?: ', Button_Switch_Keyboard:SW_Cherry_MX_1.00u_PCB, symbol Switch:SW_Push
- added SW?: A, Button_Switch_Keyboard:SW_Cherry_MX_1.00u_PCB, symbol Switch:SW_Push
- added SW?: N, Button_Switch_Keyboard:SW_Cherry_MX_1.00u_PCB, symbol Switch:SW_Push
- added SW?: C, Button_Switch_Keyboard:SW_Cherry_MX_1.00u_PCB, symbol Switch:SW_Push
- added SW?: 0, Button_Switch_Keyboard:SW_Cherry_MX_1.00u_PCB, symbol Switch:SW_Push
- added SW?: Y, Button_Switch_Keyboard:SW_Cherry_MX_1.00u_PCB, symbol Switch:SW_Push
- added SW?: ., Button_Switch_Keyboard:SW_Cherry_MX_1.00u_PCB, symbol Switch:SW_Push
- added SW?: L, Button_Switch_Keyboard:SW_Cherry_MX_1.00u_PCB, symbol Switch:SW_Push
- added SW?: Q, Button_Switch_Keyboard:SW_Cherry_MX_1.00u_PCB, symbol Switch:SW_Push
- added SW?: RotaryEncoder, symbol Device:RotaryEncoder
- added SW?: 6, Button_Switch_Keyboard:SW_Cherry_MX_1.00u_PCB, symbol Switch:SW_Push
- added SW?: B, Button_Switch_Keyboard:SW_Cherry_MX_1.00u_PCB, symbol Switch:SW_Push
Connections:
- new net: D?.2 (A), SW?.2 (x61)
- new net: R?.2, R?.2, SW?.A
- new net: C?.2, R?.2
- new net: C?.2, R?.1
- new net: R?.1, R?.2, SW?.B
- new net +3V3: R?.1, R?.1
- new net GND: C?.1, C?.1
- new net VOLUME: SW?.C
- new net X0: SW?.1, SW?.1, SW?.1, SW?.1, SW?.1, SW?.1, SW?.1, SW?.1, SW?.1, SW?.1, SW?.1, SW?.1, SW?.1, SW?.1
- new net X1: SW?.1, SW?.1, SW?.1, SW?.1, SW?.1, SW?.1, SW?.1, SW?.1, SW?.1, SW?.1, SW?.1, SW?.1, SW?.1, SW?.1
- new net X2: SW?.1, SW?.1, SW?.1, SW?.1, SW?.1, SW?.1, SW?.1, SW?.1, SW?.1, SW?.1, SW?.1, SW?.1, SW?.1
- new net X3: SW?.1, SW?.1, SW?.1, SW?.1, SW?.1, SW?.1, SW?.1, SW?.1, SW?.1, SW?.1, SW?.1, SW?.1, SW?.1
- new net X4: SW?.1, SW?.1, SW?.1, SW?.1, SW?.1, SW?.1, SW?.1
- new net Y0: D?.1 (K), D?.1 (K), D?.1 (K), D?.1 (K)
- new net Y1: D?.1 (K), D?.1 (K), D?.1 (K)
- new net Y10: D?.1 (K), D?.1 (K), D?.1 (K), D?.1 (K), D?.1 (K)
- new net Y11: D?.1 (K), D?.1 (K), D?.1 (K), D?.1 (K), D?.1 (K)
- new net Y12: D?.1 (K), D?.1 (K), D?.1 (K), D?.1 (K), D?.1 (K)
- new net Y13: D?.1 (K), D?.1 (K)
- new net Y14: D?.1 (K), D?.1 (K), D?.1 (K)
- new net Y2: D?.1 (K), D?.1 (K), D?.1 (K), D?.1 (K)
- new net Y3: D?.1 (K), D?.1 (K), D?.1 (K), D?.1 (K), D?.1 (K)
- new net Y4: D?.1 (K), D?.1 (K), D?.1 (K), D?.1 (K)
- new net Y5: D?.1 (K), D?.1 (K), D?.1 (K), D?.1 (K)
- new net Y6: D?.1 (K), D?.1 (K), D?.1 (K), D?.1 (K)
- new net Y7: D?.1 (K), D?.1 (K), D?.1 (K), D?.1 (K), D?.1 (K)
- new net Y8: D?.1 (K), D?.1 (K), D?.1 (K), D?.1 (K)
- new net Y9: D?.1 (K), D?.1 (K), D?.1 (K), D?.1 (K)
