File: switches.kicad_sch (KiCad schematic)
At the start: 129 parts

Commit message: Update layout
Connections:
- net Y12: no longer D?.1 (K)
- net Y13: now also D?.1 (K)
Other:
- moved on the sheet: D?, SW?
Changed lines of the file:
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@@
   (junction (at 248.92 81.28) (diameter 0) (color 0 0 0 0)
   )
+  (junction (at 265.43 105.41) (diameter 0) (color 0 0 0 0)
+  )
   (junction (at 123.19 105.41) (diameter 0) (color 0 0 0 0)
   )
@@
   (junction (at 88.9 109.22) (diameter 0) (color 0 0 0 0)
   )
-  (junction (at 247.65 119.38) (diameter 0) (color 0 0 0 0)
-  )
   (junction (at 213.36 81.28) (diameter 0) (color 0 0 0 0)
   )
@@
     (stroke (width 0) (type default) (color 0 0 0 0))
   )
-  (wire (pts (xy 247.65 119.38) (xy 247.65 133.35))
-    (stroke (width 0) (type default) (color 0 0 0 0))
-  )
   (wire (pts (xy 247.65 91.44) (xy 247.65 105.41))
     (stroke (width 0) (type default) (color 0 0 0 0))
@@
     (stroke (width 0) (type default) (color 0 0 0 0))
   )
-  (wire (pts (xy 247.65 133.35) (xy 246.38 133.35))
+  (wire (pts (xy 265.43 133.35) (xy 264.16 133.35))
     (stroke (width 0) (type default) (color 0 0 0 0))
   )
@@
     (stroke (width 0) (type default) (color 0 0 0 0))
   )
+  (wire (pts (xy 265.43 105.41) (xy 265.43 133.35))
+    (stroke (width 0) (type default) (color 0 0 0 0))
+  )
   (wire (pts (xy 105.41 105.41) (xy 104.14 105.41))
     (stroke (width 0) (type default) (color 0 0 0 0))
@@
     (stroke (width 0) (type default) (color 0 0 0 0))
   )
-  (wire (pts (xy 231.14 133.35) (xy 231.14 123.19))
+  (wire (pts (xy 248.92 133.35) (xy 248.92 123.19))
     (stroke (width 0) (type default) (color 0 0 0 0))
   )
@@
     (stroke (width 0) (type default) (color 0 0 0 0))
   )
-  (wire (pts (xy 213.36 123.19) (xy 231.14 123.19))
+  (wire (pts (xy 213.36 123.19) (xy 248.92 123.19))
     (stroke (width 0) (type default) (color 0 0 0 0))
   )
@@
     (pin "2")
   )
-  (symbol (lib_id "Switch:SW_Push") (at 236.22 133.35 0) (unit 1)
-    (in_bom yes) (on_board yes) (fields_autoplaced)
-    (property "Reference" "SW?" (id 0) (at 236.22 125.73 0))
-    (property "Value" ">" (id 1) (at 236.22 128.27 0))
-    (property "Footprint" "Button_Switch_Keyboard:SW_Cherry_MX_1.00u_PCB" (id 2) (at 236.22 128.27 0)
-      (effects (font (size 1.27 1.27)) hide)
-    )
-    (property "Datasheet" "~" (id 3) (at 236.22 128.27 0)
-      (effects (font (size 1.27 1.27)) hide)
-    )
-    (property "Basic Part" "Yes" (id 4) (at 236.22 133.35 0)
-      (effects (font (size 1.27 1.27)) hide)
-    )
-    (property "LCSC part number" "C318884" (id 5) (at 236.22 133.35 0)
-      (effects (font (size 1.27 1.27)) hide)
-    )
-    (property "Price" "" (id 6) (at 236.22 133.35 0)
+  (symbol (lib_id "Switch:SW_Push") (at 254 133.35 0) (unit 1)
+    (in_bom yes) (on_board yes) (fields_autoplaced)
+    (property "Reference" "SW?" (id 0) (at 254 125.73 0))
+    (property "Value" ">" (id 1) (at 254 128.27 0))
+    (property "Footprint" "Button_Switch_Keyboard:SW_Cherry_MX_1.00u_PCB" (id 2) (at 254 128.27 0)
+      (effects (font (size 1.27 1.27)) hide)
+    )
+    (property "Datasheet" "~" (id 3) (at 254 128.27 0)
+      (effects (font (size 1.27 1.27)) hide)
+    )
+    (property "Basic Part" "Yes" (id 4) (at 254 133.35 0)
+      (effects (font (size 1.27 1.27)) hide)
+    )
+    (property "LCSC part number" "C318884" (id 5) (at 254 133.35 0)
+      (effects (font (size 1.27 1.27)) hide)
+    )
+    (property "Price" "" (id 6) (at 254 133.35 0)
       (effects (font (size 1.27 1.27)) hide)
     )
@@
     (pin "2")
   )
-  (symbol (lib_id "Device:D_Small") (at 243.84 133.35 180) (unit 1)
+  (symbol (lib_id "Device:D_Small") (at 261.62 133.35 180) (unit 1)
     (in_bom yes) (on_board yes)
-    (property "Reference" "D?" (id 0) (at 243.84 127 0))
-    (property "Value" "LL4148" (id 1) (at 243.84 129.54 0))
-    (property "Footprint" "Diode_SMD:D_MiniMELF" (id 2) (at 243.84 133.35 90)
-      (effects (font (size 1.27 1.27)) hide)
-    )
-    (property "Datasheet" "~" (id 3) (at 243.84 133.35 90)
-      (effects (font (size 1.27 1.27)) hide)
-    )
-    (property "Basic Part" "Yes" (id 4) (at 243.84 133.35 0)
-      (effects (font (size 1.27 1.27)) hide)
-    )
-    (property "LCSC part number" "C9808" (id 5) (at 243.84 133.35 0)
-      (effects (font (size 1.27 1.27)) hide)
-    )
+    (property "Reference" "D?" (id 0) (at 261.62 127 0))
+    (property "Value" "LL4148" (id 1) (at 261.62 129.54 0))
+    (property "Footprint" "Diode_SMD:D_MiniMELF" (id 2) (at 261.62 133.35 90)
+      (effects (font (size 1.27 1.27)) hide)
+    )
+    (property "Datasheet" "~" (id 3) (at 261.62 133.35 90)
+      (effects (font (size 1.27 1.27)) hide)
+    )
+    (property "Basic Part" "Yes" (id 4) (at 261.62 133.35 0)
+      (effects (font (size 1.27 1.27)) hide)
+    )
+    (property "LCSC part number" "C9808" (id 5) (at 261.62 133.35 0)
+      (effects (font (size 1.27 1.27)) hide)
+    )
